File: pcb/srambo_1.sch (KiCad schematic (older format))
At the start: 29 parts, among them P1 JTAG, P10 EMMU_LEFT, P11 MMU_LEFT, P12 DRAM_RIGHT, P13 EMMU_RIGHT, P14 MMU_RIGHT, P2 GND, P3 AUX_B, P4 AUX_A, P5 DATA5-7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

Commit message: PCB: Update symbols
Parts:
- D1: symbol LED -> LED-RESCUE-srambo_1
Changed lines of the file:
@@
 EESchema Schematic File Version 2
+LIBS:srambo_1-rescue
 LIBS:power
 LIBS:device
@@
 $EndComp
 $Comp
-L LED D1
+L LED-RESCUE-srambo_1 D1
 U 1 1 57C00172
 P 5550 5450
